File: metroBlindDriver kicad/metroBlindDriver.kicad_pcb (KiCad board)
At the start: 2 copper layers, 15 parts, among them J1 12V_in, J2 SS Relais, J3 marquee_bottom_row, J4 marquee_top_row, U1 LM350_TO3

Commit message: updated pcb design
Parts:
- removed RR1: 1k, Resistor_THT:R_Axial_DIN0207_L6.3mm_D2.5mm_P7.62mm_Horizontal
- removed RR2: 330, Resistor_THT:R_Axial_DIN0207_L6.3mm_D2.5mm_P7.62mm_Horizontal
- added D1: LED, LED_THT:LED_D3.0mm, F.Cu at (100.5, 51.0)
- added K1: out relais, Relay_THT:Relay_SPST_SANYOU_SRD_Series_Form_A, F.Cu at (70.5, 44.1)
- added SW1: SW_MEC_5E, Button_Switch_THT:SW_Push_2P1T_Toggle_CK_PVA1xxH1xxxxxxV2, F.Cu at (86.5, 30.0)
- added led1: 1k, Resistor_THT:R_Axial_DIN0207_L6.3mm_D2.5mm_P7.62mm_Horizontal, F.Cu at (92.5, 44.0)
- added pd_sw_1: 1k, Resistor_THT:R_Axial_DIN0207_L6.3mm_D2.5mm_P7.62mm_Horizontal, F.Cu at (85.0, 50.5)
- J2: value SS Relais -> 220V
- J3: value marquee_bottom_row -> blind_pins_bottom_row
- J4: value marquee_top_row -> blind_pins_top_row
- U1: value LM350_TO3 -> LM7805; footprint Package_TO_SOT_THT:TO-92 -> Package_TO_SOT_THT:TO-220-3_Vertical
- tr_3: value S8050 -> S8550
- moved CRI1 83.0 mm to (35.5, 26.5), turned to -90 degrees
- moved U1 80.7 mm to (42.0, 27.9), turned to 0 degrees
- moved J2 78.9 mm to (104.0, 30.5), turned to -90 degrees
- moved CRO1 73.0 mm to (53.0, 26.5), turned to -90 degrees
- moved J1 72.9 mm to (28.5, 27.5), turned to -90 degrees
- moved pd_any_on1 59.0 mm to (78.5, 61.9)
- moved tr_1 54.6 mm to (86.5, 59.0), turned to -90 degrees
- moved r_enable_signal1 52.2 mm to (94.6, 56.9)
- moved r_run_signal1 48.7 mm to (79.0, 56.8), turned to 90 degrees
- moved tr_3 48.7 mm to (101.8, 58.7), turned to -90 degrees
- moved J4 28.7 mm to (31.0, 46.5)
- moved Arduino1 21.6 mm to (67.6, 54.3)
- moved J3 16.8 mm to (56.0, 46.5)
Connections:
- Arduino1 pad 1: unconnected-(Arduino1-D1/TX-Pad1) -> Net-(Arduino1-D1/TX)
- Arduino1 pad 13: unconnected-(Arduino1-D10-Pad13) -> Net-(Arduino1-D0/RX)
- Arduino1 pad 14: Net-(Arduino1-D11) -> unconnected-(Arduino1-D11-Pad14)
- Arduino1 pad 16: unconnected-(Arduino1-D13-Pad16) -> Net-(Arduino1-D13)
- Arduino1 pad 2: unconnected-(Arduino1-D0/RX-Pad2) -> Net-(Arduino1-D0/RX)
- J2 pad 2: GND -> Net-(J2-Pin_2)
- J4 pad 3: Net-(Arduino1-D11) -> Net-(Arduino1-D0/RX)
- U1 pad 1: Net-(U1-ADJ) -> +12C
- U1 pad 2: +12C -> GND
- pd_any_on1 pad 1: Net-(Arduino1-D11) -> Net-(Arduino1-D0/RX)
- r_run_signal1 pad 1: Net-(Arduino1-D11) -> Net-(Arduino1-D0/RX)
- tr_1 pad 1: Net-(J2-Pin_1) -> Net-(tr_1-E)
Routing:
- net Net-(Arduino1-D11): track 103.6 -> 0.00 mm
- net Net-(Arduino1-D13): track 0.00 -> 94.0 mm
- net GND: track 224.8 -> 138.1 mm
- net Net-(Arduino1-D0/RX): track 0.00 -> 60.0 mm
- net Net-(Arduino1-D12): track 8.77 -> 66.9 mm
- net Net-(Arduino1-D1/TX): track 0.00 -> 42.2 mm
- net Net-(J2-Pin_2): track 0.00 -> 39.8 mm
- net +5V: track 130.4 -> 97.5 mm
- net Net-(Arduino1-D8): track 31.8 -> 8.24 mm
- net Net-(tr_1-E): track 0.00 -> 20.9 mm
- net Net-(U1-ADJ): track 17.8 -> 0.00 mm
- net Net-(tr_3-B): track 25.0 -> 8.40 mm
- net Net-(J2-Pin_1): track 15.9 -> 32.2 mm
- net Net-(tr_1-B): track 48.1 -> 34.4 mm
- net Net-(D1-K): track 0.00 -> 10.9 mm
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Other:
- board outline added: 83.5 x 49.5 mm
