File: metroBlindDriver kicad/metroBlindDriver.kicad_sch (KiCad schematic)
At the start: 15 parts, among them J1 12V_in, J2 SS Relais, J3 marquee_bottom_row, J4 marquee_top_row, U1 LM350_TO3

Commit message: updated pcb design
Parts:
- removed RR1: 1k, Resistor_THT:R_Axial_DIN0207_L6.3mm_D2.5mm_P7.62mm_Horizontal, symbol Device:R
- removed RR2: 330, Resistor_THT:R_Axial_DIN0207_L6.3mm_D2.5mm_P7.62mm_Horizontal, symbol Device:R
- added D1: LED, LED_THT:LED_D3.0mm, symbol Device:LED
- added K1: out relais, Relay_THT:Relay_SPST_SANYOU_SRD_Series_Form_A, symbol Relay:SANYOU_SRD_Form_A
- added SW1: SW_MEC_5E, Button_Switch_THT:SW_Push_2P1T_Toggle_CK_PVA1xxH1xxxxxxV2, symbol Switch:SW_MEC_5E
- added led1, pd_sw_1: 1k, Resistor_THT:R_Axial_DIN0207_L6.3mm_D2.5mm_P7.62mm_Horizontal, symbol Device:R
- J2: value SS Relais -> 220V
- J3: value marquee_bottom_row -> blind_pins_bottom_row
- J4: value marquee_top_row -> blind_pins_top_row
- U1: value LM350_TO3 -> LM7805; footprint Package_TO_SOT_THT:TO-92 -> Package_TO_SOT_THT:TO-220-3_Vertical; symbol Regulator_Linear:LM350_TO3 -> Regulator_Linear:LM78M05_TO220
- tr_3: value S8050 -> S8550
Connections:
- net +12C: now also U1.1 (VI); no longer U1.2 (VI)
- net +5V: now also SW1.3 (K)
- net GND: now also U1.2 (GND), K1.5, led1.2, pd_sw_1.2; no longer J2.2 (Pin_2)
- net at J4.3 (Pin_3), pd_any_on1.1, r_run_signal1.1: now also Arduino1.13 (D10), Arduino1.2 (D0/RX); no longer Arduino1.14 (D11)
- net at tr_1.1 (E): now also K1.2; no longer J2.1 (Pin_1)
- net at Arduino1.1 (D1/TX): now also SW1.2, pd_sw_1.1
- net at Arduino1.16 (D13): now also D1.2 (A)
- new net: D1.1 (K), led1.1
- new net: J2.1 (Pin_1), K1.3
- new net: J2.2 (Pin_2), K1.1
Other:
- moved on the sheet: J1, J2, r_enable_signal1, tr_3
